Commit message: Add sensor tower assembly, reassigned LIDAR sensor origin

File: husky/husky_description/urdf/husky.urdf.xacro (robot description, xacro)
@@ -41,34 +41,4 @@
     </gazebo>
   </xacro:if>
-  <!-- ZED Camera -->
-  <link name="zed_link">
-    <visual>
-      <origin xyz="0 0 0" rpy="0 0 0"/>
-      <geometry>
-        <box size="0.175 0.033 0.03"/>
-      </geometry>
-    </visual>
-    <collision>
-      <geometry>
-        <box size="0.175 0.033 0.03"/>
-      </geometry>
-    </collision>
-    <inertial>
-      <mass value="0.16"/>
-      <inertia ixx="0.001" ixy="0" ixz="0"
-               iyy="0.001" iyz="0" izz="0.001"/>
-    </inertial>
-  </link>
-  <joint name="zed_joint" type="fixed">
-    <parent link="base_link"/>
-    <child link="zed_link"/>
-    <origin xyz="0.2 0.0 0.15" rpy="0 0 0"/>
-  </joint>
-  <link name="zed_optical_frame"/>
-  <joint name="zed_optical_joint" type="fixed">
-    <parent link="zed_link"/>
-    <child link="zed_optical_frame"/>
-    <origin xyz="0 0 0" rpy="-1.5708 0 -1.5708"/>
-  </joint>
   <!-- Double Rail Right-->
   <link name="double_rail_link_right">
@@ -171,32 +141,45 @@
     <origin xyz="-0.203 -0.2095 0.35" rpy="1.570796327 1.570796327 -1.570796327"/>
   </joint>
-  <!-- OS1 LIDAR -->
-  <link name="os1_lidar_link">
-    <visual>
-      <origin xyz="0 0 0" rpy="1.570796327 0 0"/>
-      <geometry>
-        <mesh filename="package://husky_description/meshes/LIDAR.STL"/>
-      </geometry>
-    </visual>
-    <collision>
-      <geometry>
-        <mesh filename="package://husky_description/meshes/LIDAR.STL"/>
-      </geometry>
-    </collision>
-    <inertial>
-      <mass value="0.447"/>
-      <inertia ixx="0.005" ixy="0" ixz="0"
-               iyy="0.0002" iyz="0" izz="0.0005"/>
-    </inertial>
-  </link>
-  <joint name="os1_lidar_joint" type="fixed">
+  <!-- Sensor Box -->
+  <link name="sensor_box_link">
+    <visual>
+      <origin xyz="0 0 0" rpy="0 0 0"/>
+      <geometry>
+        <mesh filename="package://husky_description/meshes/SensorBox.STL"/>
+      </geometry>
+    </visual>
+    <collision>
+      <geometry>
+        <mesh filename="package://husky_description/meshes/SensorBox.STL"/>
+      </geometry>
+    </collision>
+    <inertial>
+      <mass value="3"/>
+      <inertia ixx="0.09" ixy="0" ixz="0"
+               iyy="0.08" iyz="0.03" izz="0.03"/>
+    </inertial>
+  </link>
+  <joint name="sensor_box_joint" type="fixed">
     <parent link="double_rail_link_short"/>
-    <child link="os1_lidar_link"/>
-    <origin xyz="-0.080 0.2 0.152" rpy="1.570796327 0 3.141592654"/>
-  </joint>
-  <gazebo reference="os1_lidar_link">
+    <child link="sensor_box_link"/>
+    <origin xyz="0.07 0.039 0.4025" rpy="-1.570796327 1.570796327 0"/>
+  </joint>
+  <!-- Invisible helper link at the actual lidar position -->
+  <link name="os1_ray_origin_link">
+    <inertial>
+      <mass value="0.001"/>
+      <inertia ixx="0.0001" ixy="0" ixz="0"
+               iyy="0.0001" iyz="0" izz="0.0001"/>
+    </inertial>
+  </link>
+  <joint name="os1_ray_origin_joint" type="fixed">
+    <parent link="sensor_box_link"/>
+    <child link="os1_ray_origin_link"/>
+    <origin xyz="0 0 0.22605" rpy="0 0 0"/>
+  </joint>
+  <gazebo reference="os1_ray_origin_link">
     <sensor type="gpu_ray" name="os1_sensor">
-      <pose>0 0 0 0  0</pose>
-      <visualize>false</visualize>
+      <pose>0 0 0 0 0 0</pose>
+      <visualize>true</visualize>
       <update_rate>10</update_rate>
       <ray>
@@ -232,5 +215,5 @@
       <sensor_name>os1_sensor</sensor_name>
       <topic_name>/ouster/points</topic_name>
-      <frame_name>os1_lidar_link</frame_name>
+      <frame_name>sensor_box_link</frame_name>
       <min_intensity>0</min_intensity>
     </plugin>
